File: hardware/irondriver.sch (KiCad schematic (older format))
At the start: 71 parts, among them P1 CONN_01X02, P2 CONN_01X02, P3 CONN_02X07, P6 CONN_01X03, Q1 MMBT3906, Q2 MMBT3904, Q3 MMBT3904, U1 STM32F103C8T6, U2 LM2596, U3 AD8606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

Commit message: Changed silk placement and size. Added logo and author information.
Parts:
- L1: footprint Inductors:SELF-WE-PD-XXL -> Inductors:SELF-WE-PD3S
Changed lines of the file:
@@
 F 0 "L1" H 4630 1640 50  0000 L CNN
 F 1 "1mH" H 4630 1560 50  0000 L CNN
-F 2 "Inductors:SELF-WE-PD-XXL" H 4600 1600 50  0001 C CNN
+F 2 "Inductors:SELF-WE-PD3S" H 4600 1600 50  0001 C CNN
 F 3 "" H 4600 1600 50  0000 C CNN
 	1    4600 1600
